File: hardware/analog-front-end/PC_Interstage.kicad_pcb (KiCad board)
At the start: 2 copper layers, 82.6 x 14.3 mm, 32 parts, among them IC1 OPA1678IDR, J1 Conn_01x04_Socket, J2 Conn_01x01_Socket, J3 Conn_01x01_Socket, J4 Conn_01x01_Socket, J5 Conn_01x01_Socket, J6 Conn_01x04_Socket, J7 Conn_01x04_Socket, J8 Conn_01x04_Socket, J9 Conn_01x04_Socket, U1 REF3012

Commit message: fix inconsistency
Parts:
- C1: value 2.2p -> 1p
- C10: value 4.7p -> 100p
- C3: value 100p -> INF
- C6: value 10u -> 0
- D1: footprint SamacSys_Parts:S1223-01 -> Mouser Lib:S1223-01
- IC1: value OPA1678IDR -> OPA2354
- R3: value 100K -> INF
- R4: value 5K -> 3.3k
- R6: value 10 -> 0
- R7: value 0 -> 15k
- R8: value 10G -> 10k
Changed lines of the file:
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@@
 		(property ki_fp_filters "R_*")
 		(sheetname "/")
-		(sheetfile "SUCHAI Interstage Dual Camera.kicad_sch")
+		(sheetfile "PC_Interstage.kicad_sch")
 		(attr smd)
 		(fp_line
@@
 			)
 		)
-		(property "Value" "10"
+		(property "Value" "0"
 			(at 0 1.65 0)
 			(layer "F.Fab")
@@
 		(property ki_fp_filters "R_*")
 		(sheetname "/")
-		(sheetfile "SUCHAI Interstage Dual Camera.kicad_sch")
+		(sheetfile "PC_Interstage.kicad_sch")
 		(attr smd)
 		(fp_line
@@
 		(property ki_fp_filters "R_*")
 		(sheetname "/")
-		(sheetfile "SUCHAI Interstage Dual Camera.kicad_sch")
+		(sheetfile "PC_Interstage.kicad_sch")
 		(attr smd)
 		(fp_line
@@
 		(property ki_fp_filters "SOT?23*")
 		(sheetname "/")
-		(sheetfile "SUCHAI Interstage Dual Camera.kicad_sch")
+		(sheetfile "PC_Interstage.kicad_sch")
 		(attr smd)
 		(fp_line
@@
 		(property ki_fp_filters "C_*")
 		(sheetname "/")
-		(sheetfile "SUCHAI Interstage Dual Camera.kicad_sch")
+		(sheetfile "PC_Interstage.kicad_sch")
 		(attr smd)
 		(fp_line
@@
 		(property ki_fp_filters "C_*")
 		(sheetname "/")
-		(sheetfile "SUCHAI Interstage Dual Camera.kicad_sch")
+		(sheetfile "PC_Interstage.kicad_sch")
 		(attr smd)
 		(fp_line
@@
 			)
 		)
-		(property "Value" "4.7p"
+		(property "Value" "100p"
 			(at 0 1.68 90)
 			(layer "F.Fab")
@@
 		(property ki_fp_filters "C_*")
 		(sheetname "/")
-		(sheetfile "SUCHAI Interstage Dual Camera.kicad_sch")
+		(sheetfile "PC_Interstage.kicad_sch")
 		(attr smd)
 		(fp_line
@@
 		(property ki_fp_filters "Connector*:*_1x??_*")
 		(sheetname "/")
-		(sheetfile "SUCHAI Interstage Dual Camera.kicad_sch")
+		(sheetfile "PC_Interstage.kicad_sch")
 		(attr through_hole)
 		(fp_line
@@
 		(property ki_fp_filters "C_*")
 		(sheetname "/")
-		(sheetfile "SUCHAI Interstage Dual Camera.kicad_sch")
+		(sheetfile "PC_Interstage.kicad_sch")
 		(attr smd)
 		(fp_line
@@
 		(property ki_fp_filters "Connector*:*_1x??_*")
 		(sheetname "/")
-		(sheetfile "SUCHAI Interstage Dual Camera.kicad_sch")
+		(sheetfile "PC_Interstage.kicad_sch")
 		(attr through_hole)
 		(fp_line
@@
 		(property ki_fp_filters "Connector*:*_1x??_*")
 		(sheetname "/")
-		(sheetfile "SUCHAI Interstage Dual Camera.kicad_sch")
+		(sheetfile "PC_Interstage.kicad_sch")
 		(attr through_hole)
 		(fp_line
@@
 		(property ki_fp_filters "C_*")
 		(sheetname "/")
-		(sheetfile "SUCHAI Interstage Dual Camera.kicad_sch")
+		(sheetfile "PC_Interstage.kicad_sch")
 		(attr smd)
 		(fp_line
@@
 			)
 		)
-		(property "Value" "5K"
+		(property "Value" "3.3k"
 			(at 0 1.65 0)
 			(layer "F.Fab")
@@
 		(property ki_fp_filters "R_*")
 		(sheetname "/")
-		(sheetfile "SUCHAI Interstage Dual Camera.kicad_sch")
+		(sheetfile "PC_Interstage.kicad_sch")
 		(attr smd)
 		(fp_line
@@
 		(property ki_fp_filters "Connector*:*_1x??_*")
 		(sheetname "/")
-		(sheetfile "SUCHAI Interstage Dual Camera.kicad_sch")
+		(sheetfile "PC_Interstage.kicad_sch")
 		(attr smd)
 		(fp_line
@@
 			)
 		)
-		(property "Value" "0"
+		(property "Value" "15k"
 			(at 0 1.65 90)
 			(layer "F.Fab")
@@
 		(property ki_fp_filters "R_*")
 		(sheetname "/")
-		(sheetfile "SUCHAI Interstage Dual Camera.kicad_sch")
+		(sheetfile "PC_Interstage.kicad_sch")
 		(attr smd)
 		(fp_line
@@
 			)
 		)
-		(property "Value" "10G"
+		(property "Value" "10k"
 			(at 0 1.65 90)
 			(layer "F.Fab")
@@
 		(property ki_fp_filters "R_*")
 		(sheetname "/")
-		(sheetfile "SUCHAI Interstage Dual Camera.kicad_sch")
+		(sheetfile "PC_Interstage.kicad_sch")
 		(attr smd)
 		(fp_line
@@
 		(property ki_fp_filters "Connector*:*_1x??_*")
 		(sheetname "/")
-		(sheetfile "SUCHAI Interstage Dual Camera.kicad_sch")
+		(sheetfile "PC_Interstage.kicad_sch")
 		(attr smd)
 		(fp_line
@@
 		(property ki_fp_filters "Connector*:*_1x??_*")
 		(sheetname "/")
-		(sheetfile "SUCHAI Interstage Dual Camera.kicad_sch")
+		(sheetfile "PC_Interstage.kicad_sch")
 		(attr through_hole)
 		(fp_line
@@
 		(property ki_fp_filters "R_*")
 		(sheetname "/")
-		(sheetfile "SUCHAI Interstage Dual Camera.kicad_sch")
+		(sheetfile "PC_Interstage.kicad_sch")
 		(attr smd)
 		(fp_line
@@
 			)
 		)
-		(property "Value" "100K"
+		(property "Value" "INF"
 			(at 0 1.65 90)
 			(layer "F.Fab")
@@
 		(property ki_fp_filters "R_*")
 		(sheetname "/")
-		(sheetfile "SUCHAI Interstage Dual Camera.kicad_sch")
+		(sheetfile "PC_Interstage.kicad_sch")
 		(attr smd)
 		(fp_line
@@
 		(property ki_fp_filters "R_*")
 		(sheetname "/")
-		(sheetfile "SUCHAI Interstage Dual Camera.kicad_sch")
+		(sheetfile "PC_Interstage.kicad_sch")
 		(attr smd)
 		(fp_line
@@
 			)
 		)
-		(property "Value" "2.2p"
+		(property "Value" "1p"
 			(at 0 1.68 0)
 			(layer "F.Fab")
@@
 		(property ki_fp_filters "C_*")
 		(sheetname "/")
-		(sheetfile "SUCHAI Interstage Dual Camera.kicad_sch")
+		(sheetfile "PC_Interstage.kicad_sch")
 		(attr smd)
 		(fp_line
@@
 		(property ki_fp_filters "C_*")
 		(sheetname "/")
-		(sheetfile "SUCHAI Interstage Dual Camera.kicad_sch")
+		(sheetfile "PC_Interstage.kicad_sch")
 		(attr smd)
 		(fp_line
@@
 		(property ki_fp_filters "C_*")
 		(sheetname "/")
-		(sheetfile "SUCHAI Interstage Dual Camera.kicad_sch")
+		(sheetfile "PC_Interstage.kicad_sch")
 		(attr smd)
 		(fp_line
@@
 			)
 		)
-		(property "Value" "OPA1678IDR"
+		(property "Value" "OPA2354"
 			(at 0 0 0)
 			(layer "F.SilkS")
@@
 		)
 		(sheetname "/")
-		(sheetfile "SUCHAI Interstage Dual Camera.kicad_sch")
+		(sheetfile "PC_Interstage.kicad_sch")
 		(attr smd)
 		(fp_line
@@
 		(property ki_fp_filters "Connector*:*_1x??_*")
 		(sheetname "/")
-		(sheetfile "SUCHAI Interstage Dual Camera.kicad_sch")
+		(sheetfile "PC_Interstage.kicad_sch")
 		(attr through_hole)
 		(fp_line
@@
 		)
 	)
-	(footprint "SamacSys_Parts:S1223-01"
+	(footprint "Mouser Lib:S1223-01"
 		(layer "F.Cu")
 		(at 149.16 98.46)
@@
 		)
 		(sheetname "/")
-		(sheetfile "SUCHAI Interstage Dual Camera.kicad_sch")
+		(sheetfile "PC_Interstage.kicad_sch")
 		(attr through_hole)
 		(fp_line
@@
 		(property ki_fp_filters "Connector*:*_1x??_*")
 		(sheetname "/")
-		(sheetfile "SUCHAI Interstage Dual Camera.kicad_sch")
+		(sheetfile "PC_Interstage.kicad_sch")
 		(attr smd)
 		(fp_line
@@
 			)
 		)
-		(property "Value" "10u"
+		(property "Value" "0"
 			(at 0 -1.68 0)
 			(layer "B.Fab")
@@
 		(property ki_fp_filters "C_*")
 		(sheetname "/")
-		(sheetfile "SUCHAI Interstage Dual Camera.kicad_sch")
+		(sheetfile "PC_Interstage.kicad_sch")
 		(attr smd)
 		(fp_line
@@
 		(property ki_fp_filters "R_*")
 		(sheetname "/")
-		(sheetfile "SUCHAI Interstage Dual Camera.kicad_sch")
+		(sheetfile "PC_Interstage.kicad_sch")
 		(attr smd)
 		(fp_line
@@
 		(property ki_fp_filters "Connector*:*_1x??_*")
 		(sheetname "/")
-		(sheetfile "SUCHAI Interstage Dual Camera.kicad_sch")
+		(sheetfile "PC_Interstage.kicad_sch")
 		(attr smd)
 		(fp_line
@@
 			)
 		)
-		(property "Value" "100p"
+		(property "Value" "INF"
 			(at 0 -1.68 90)
 			(layer "B.Fab")
@@
 		(property ki_fp_filters "C_*")
 		(sheetname "/")
-		(sheetfile "SUCHAI Interstage Dual Camera.kicad_sch")
+		(sheetfile "PC_Interstage.kicad_sch")
 		(attr smd)
 		(fp_line
